Commit message: Modified URDF

File: omni_drive_arduino/description/ros2_control/omnibot.ros2_control.xacro (robot description, xacro)
@@ -11,5 +11,5 @@
         <param name="device">/dev/ttyACM0</param>
         <param name="baud_rate">9600</param>
-        <param name="timeout_ms">500</param>
+        <param name="timeout_ms">1000</param>
       </hardware>
       <joint name="${prefix}first_wheel_joint">

File: omni_drive_arduino/description/urdf/omnibot.materials.xacro (robot description, xacro)
@@ -4,3 +4,6 @@
     <color rgba="0.700 0.700 0.700 1.000"/>
   </material>
+  <material name="black">
+    <color rgba="0.000 0.000 0.000 1.000"/>
+  </material>
 </robot>

File: omni_drive_arduino/description/urdf/omnibot.urdf.xacro (robot description, xacro)
@@ -4,9 +4,9 @@
   <xacro:arg name="prefix" default="" />
   <!-- Import urdf description -->
-  <xacro:include filename="$(find omni_drive_arduino)/urdf/diffbot_description.urdf.xacro" />
+  <xacro:include filename="$(find omni_drive_arduino)/urdf/omnibot_description.urdf.xacro" />
   <!-- Import Rviz colors -->
-  <xacro:include filename="$(find omni_drive_arduino)/urdf/diffbot.materials.xacro" />
-  <!-- Import diffbot ros2_control description -->
-  <xacro:include filename="$(find omni_drive_arduino)/ros2_control/diffbot.ros2_control.xacro" />
+  <xacro:include filename="$(find omni_drive_arduino)/urdf/omnibot.materials.xacro" />
+  <!-- Import omnibot ros2_control description -->
+  <xacro:include filename="$(find omni_drive_arduino)/ros2_control/omnibot.ros2_control.xacro" />
   <xacro:omnibot prefix="$(arg prefix)" />
   <xacro:omnibot_ros2_control
